Commit message: Arreglo en las rutas de las mallas

File: urdf/px_collision.urdf (robot description, URDF)
Before this commit: robot px_robot, 7 links, 6 joints
Links:
- link base_link: geometry collision mesh filename=package://px_robot/meshes/Base.STL scale=1 1 1; visual mesh filename=package://px_robot/meshes/Base.STL scale=1 1 1
- link link1: geometry collision mesh filename=package://px_robot/meshes/Shoulder.STL scale=1 1 1; visual mesh filename=package://px_robot/meshes/Shoulder.STL scale=1 1 1
- link link2: geometry collision mesh filename=package://px_robot/meshes/Bicep.STL scale=1 1 1; visual mesh filename=package://px_robot/meshes/Bicep.STL scale=1 1 1
- link link3: geometry collision mesh filename=package://px_robot/meshes/Bicep.STL scale=1 1 1; visual mesh filename=package://px_robot/meshes/Bicep.STL scale=1 1 1
- link link4: geometry collision mesh filename=package://px_robot/meshes/Wrist.STL scale=1 1 1; visual mesh filename=package://px_robot/meshes/Wrist.STL scale=1 1 1
